File: Hardware/Cube-Breakout-Board/Cube-Breakout-Board.kicad_sch (KiCad schematic)
At the start: 4 parts, among them J1 Conn_01x22, J2 Conn_01x30, J3 Pixhawk_Cube_DF17_80_Pin_Grou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, J4 Conn_01x30

Commit message: Finished routing, board sizing, silkscreen text
Parts:
- added J2: Pixhawk_Cube_DF17_80_Pin_Grouped, libraries:Cube_DF17_Mount, symbol CubeCarrierBoard:Pixhawk_Cube_DF17_80_Pin_Grouped_Bottom
- renumbered J3 to J1, J4 to J3, J1 to J4, J2 to J5
Connections:
- net ALARM: now also J2.23 (ALARM)
- net AUX_BATT_CURRENT_SENS: now also J2.26 (AUX_BATT_CURRENT_SENS)
- net AUX_BATT_VOLTAGE_SENS: now also J2.24 (AUX_BATT_VOLTAGE_SENS)
- net BATT_CURRENT_SENS_PROT: now also J2.50 (BATT_CURRENT_SENS_PROT)
- net BATT_VOLTAGE_SENS_PROT: now also J2.48 (BATT_VOLTAGE_SENS_PROT)
- net CAN_H_1: now also J2.80 (CAN_H_1)
- net CAN_H_2: now also J2.42 (CAN_H_2)
- net CAN_L_1: now also J2.78 (CAN_L_1)
- net CAN_L_2: now also J2.40 (CAL_L_2)
- net EXTERN_CS: now also J2.6 (EXTERN_CS)
- net EXTERN_DRDY: now also J2.12 (EXTERN_DRDY)
- net FMU_CH1_PROT: now also J2.49 (FMU_CH1_PROT)
- net FMU_CH2_PROT: now also J2.51 (FMU_CH2_PROT)
- net FMU_CH3_PROT: now also J2.53 (FMU_CH3_PROT)
- net FMU_CH4_PROT: now also J2.55 (FMU_CH4_PROT)
- net FMU_CH5_PROT: now also J2.57 (FMU_CH5_PROT)
- net FMU_CH6_PROT: now also J2.59 (FMU_CH6_PROT)
- net FMU_LED_AMBER: now also J2.1 (FMU_LED_AMBER)
- net FMU_SWCLK: now also J2.4 (FMU_SWCLK)
- net FMU_SWDIO: now also J2.2 (FMU_SWDIO)
- net FMU_~{RESET}: now also J2.8 (FMU_~{RESET})
- net GND: now also J1.81 (GND), J1.S1 (GND), J1.S2 (GND), J2.14 (GND), J2.16 (GND), J2.81 (GND), J2.S1 (GND), J2.S2 (GND)
- net I2C_1_SCL: now also J2.38 (I2C_1_SCL)
- net I2C_1_SDA: now also J2.36 (I2C_1_SDA)
- net I2C_2_SCL: now also J2.5 (I2C_2_SCL)
- net I2C_2_SDA: now also J2.3 (I2C_2_SDA)
- net IO_CH1_PROT: now also J2.79 (IO_CH1_PROT)
- net IO_CH2_PROT: now also J2.77 (IO_CH2_PROT)
- net IO_CH3_PROT: now also J2.75 (IO_CH3_PROT)
- net IO_CH4_PROT: now also J2.73 (IO_CH4_PROT)
- net IO_CH5_PROT: now also J2.71 (IO_CH5_PROT)
- net IO_CH6_PROT: now also J2.69 (IO_CH6_PROT)
- net IO_CH7_PROT: now also J2.67 (IO_CH7_PROT)
- net IO_CH8_PROT: now also J2.65 (IO_CH8_PROT)
- net IO_LED_SAFET_PROT: now also J2.27 (IO_LED_SAFET_PROT)
- net IO_SWCLK: now also J2.72 (IO_SWCLK)
- net IO_SWDIO: now also J2.70 (IO_SWDIO)
- net IO_USART1_RX: now also J2.47 (IO_USART1_RX_SPECTRUM_DSM)
- net IO_USART_1_TX: now also J2.45 (IO_USART_1_TX)
- net IO_VDD_3V3: now also J2.25 (IO_VDD_3V3)
- net IO_VDD_5V: now also J2.66 (IO_VDD_5V5)
- net IO_~{RESET}: now also J2.76 (IO_~{RESET})
- net OTG_DM1: now also J2.34 (OTG_DM1)
- net OTG_DP1: now also J2.32 (OTG_DP1)
- net PPM_SBUS_PROT: now also J2.61 (PPM_SBUS_PROT)
- net PRESSURE_SENS_IN: now also J2.22 (PRESSURE_SENS_IN)
- net PROT_SPARE_1: now also J2.7 (PROT_SPARE_1)
- net PROT_SPARE_2: now also J2.9 (PROT_SPARE_2)
- net S.BUS_OUT: now also J2.63 (S.BUS_OUT)
- net SAFETY: now also J2.18 (SAFETY)
- net SERIAL_1_CTS: now also J2.43 (SERIAL_1_CTS)
- net SERIAL_1_RTS: now also J2.41 (SERIAL_1_RTS)
- net SERIAL_1_RX: now also J2.37 (SERIAL_1_RX)
- net SERIAL_1_TX: now also J2.39 (SERIAL_1_TX)
- net SERIAL_2_CTS: now also J2.31 (SERIAL_2_CTS)
- net SERIAL_2_RTS: now also J2.29 (SERIAL_2_RTS)
- net SERIAL_2_RX: now also J2.33 (SERIAL_2_RX)
- net SERIAL_2_TX: now also J2.35 (SERIAL_2_TX)
- net SERIAL_3_RX: now also J2.19 (SERIAL_3_RX)
- net SERIAL_3_TX: now also J2.21 (SERIAL_3_TX)
- net SERIAL_4_RX: now also J2.15 (SERIAL_4_RX)
- net SERIAL_4_TX: now also J2.17 (SERIAL_4_TX)
- net SERIAL_5_RX: now also J2.11 (SERIAL_5_RX)
- net SERIAL_5_TX: now also J2.13 (SERIAL_5_TX)
- net SPI_EXT_MISO: now also J2.68 (SPI_EXT_MISO)
- net SPI_EXT_MOSI: now also J2.52 (SPI_EXT_MOSI)
- net SPI_EXT_SCK: now also J2.74 (SPI_EXT_SCK)
- net VBUS: now also J2.30 (VBUS)
- net VBUS_VALID: now also J2.60 (VBUS_VALID)
- net VDD_3V3_SPEKTRUM_EN: now also J2.20 (VDD_3V3_SPEKTRUM_EN)
- net VDD_5V_HIPOWER_OC: now also J2.46 (VDD_5V_HIPOWER_OC)
- net VDD_5V_IN_PROT: now also J2.62 (VDD_5V_IN_PROT), J2.64 (VDD_5V_IN_PROT)
- net VDD_5V_PERIPH_EN: now also J2.28 (VDD_5V_PERIPH_EN)
- net VDD_5V_PERIPH_OC: now also J2.44 (VDD_5V_PERIPH_OC)
- net VDD_BACKUP_VALID: now also J2.58 (VDD_BACKUP_VALID)
- net VDD_BRICK_VALID: now also J2.56 (VDD_BRICK_VALID)
- net VDD_SERVO: now also J2.54 (VDD_SERVO)
- net VDD_SERVO_IN: now also J2.10 (VDD_SERVO_IN)
Other:
- moved on the sheet: J3, J4, J5
